File: EPS/Kicad Files/charge schem/charge schem.kicad_sch (KiCad schematic)
At the start: 23 parts, among them J1 USB_C_Receptacle, U1 MAX77757JEFG435+, U2 MAX17055EWL+T

Commit message: added one piece - test
Parts:
- added U?: ADP5063, Package_DFN_QFN:QFN-20-1EP_4x4mm_P0.5mm_EP2.5x2.5mm, symbol Battery_Management:ADP5063
Connections:
- new net: U?.10 (ISO_Sx), U?.11 (ISO_Sx), U?.9 (ISO_Sx)
- new net: U?.12 (ISO_Bx), U?.13 (ISO_Bx), U?.14 (ISO_Bx)
- new net: U?.6 (VINx), U?.7 (VINx), U?.8 (VINx)
Changed lines of the file:
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@@
     (pin "S1")
+  )
+  (symbol (lib_id "Battery_Management:ADP5063") (at 46.99 151.13 0) (unit 1)
+    (in_bom yes) (on_board yes) (fields_autoplaced)
+    (property "Reference" "U?" (id 0) (at 46.99 130.81 0))
+    (property "Value" "ADP5063" (id 1) (at 46.99 133.35 0))
+    (property "Footprint" "Package_DFN_QFN:QFN-20-1EP_4x4mm_P0.5mm_EP2.5x2.5mm" (id 2) (at 53.34 173.99 0)
+      (effects (font (size 1.27 1.27)) hide)
+    )
+    (property "Datasheet" "https://www.analog.com/media/en/technical-documentation/data-sheets/ADP5063.pdf" (id 3) (at -8.89 114.3 0)
+      (effects (font (size 1.27 1.27)) hide)
+    )
+    (pin "1")
+    (pin "10")
+    (pin "11")
+    (pin "12")
+    (pin "13")
+    (pin "14")
+    (pin "15")
+    (pin "16")
+    (pin "17")
+    (pin "18")
+    (pin "19")
+    (pin "2")
+    (pin "20")
+    (pin "21")
+    (pin "3")
+    (pin "4")
+    (pin "5")
+    (pin "6")
+    (pin "7")
+    (pin "8")
+    (pin "9")
   )
   (symbol (lib_id "power:GNDPWR") (at 167.64 104.14 0) (unit 1)
@@
       (reference "U2") (unit 1) (value "MAX17055EWL+T") (footprint "17055 foot:MAX17055EWL&plus_T")
     )
-  )
+    (path "/ce4b6c19-1441-4e43-8af4-a7f34dfbb538"
+      (reference "U?") (unit 1) (value "ADP5063") (footprint "Package_DFN_QFN:QFN-20-1EP_4x4mm_P0.5mm_EP2.5x2.5mm")
+    )
+  )
