File: CD&H/CDH/cm4-gpio.kicad_sch (KiCad schematic)
At the start: 18 parts, among them J1 THD-20-R, U1 ATA6560-GAQW-VAO, U3 MCP2510-E/SO, U4 74LVC1G07SE-7

Commit message: updates
Parts:
- removed H1, H2, H3, H4: 3mm_Mounting_Hole, MountingHole:MountingHole_3mm, symbol Mechanical:MountingHole
- added P1, P2: S04B-PASK-2(LF)(SN), S04B-PASK-2_LF__SN_:JST_S04B-PASK-2(LF)(SN), symbol S04B-PASK-2_LF__SN_:S04B-PASK-2(LF)(SN)
Connections:
- net +5V: now also P1.1, P2.1
- net GND: now also P1.4, P2.4
- net GPIO12: now also P2.2; no longer U3.12 (~{INT})
- net GPIO14: now also P1.2; no longer J1.8 (Pin_8)
- net GPIO15: now also P1.3; no longer J1.10 (Pin_10)
- net GPIO13: now reaches Module2.28 (GPIO13)
- net GPIO13: now also P2.3
