File: Payload/ColoradoCUBE_Payload/ColoradoCUBE_Payload.kicad_pcb (KiCad board)
At the start: 2 copper layers, 96 x 90 mm, 56 parts, among them J1 Conn_02x20_Odd_Even, J2 Generic_Conn_01x05, J3 Conn_01x06, J4 Conn_01x04, J5 Conn_01x02, J6 Conn_01x02, J7 Conn_01x02, SW1 SW_SPST, U1 PIC18F27Q84-E/SP, U2 SHT40-AD1B-R2, U3 ATA6560-GAQW-VAO, U4 MS580502BA01-50

Commit message: updates
Parts:
- J1: value Conn_02x20_Odd_Even -> SSQ-120-03-F-D
- J2: value Generic_Conn_01x05 -> PH1-05-UA
- J3: value Conn_01x06 -> PR20206VBNN
- J4: value Conn_01x04 -> PR20204VBNN
- J5, J6: value Conn_01x02 -> PH1-02-UA
Changed lines of the file:
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@@
       (effects (font (size 1 1) (thickness 0.15)))
     )
-    (fp_text value "Conn_01x04" (at 0 9.95) (layer "F.Fab")
+    (fp_text value "PR20204VBNN" (at 0 9.95) (layer "F.Fab")
       (effects (font (size 1 1) (thickness 0.15)))
     )
@@
       (effects (font (size 1 1) (thickness 0.15)))
     )
-    (fp_text value "Conn_01x06" (at 0.508 -3.048) (layer "F.Fab")
+    (fp_text value "PR20206VBNN" (at 0.508 -3.048) (layer "F.Fab")
       (effects (font (size 1 1) (thickness 0.15)))
     )
@@
       (effects (font (size 1 1) (thickness 0.15)))
     )
-    (fp_text value "Generic_Conn_01x05" (at -2.595 4.627) (layer "F.Fab")
+    (fp_text value "PH1-05-UA" (at -2.595 4.627) (layer "F.Fab")
       (effects (font (size 1 1) (thickness 0.15)))
     )
@@
       (effects (font (size 1 1) (thickness 0.15)))
     )
-    (fp_text value "Conn_01x02" (at 0 4.87) (layer "F.Fab")
+    (fp_text value "PH1-02-UA" (at 0 4.87) (layer "F.Fab")
       (effects (font (size 1 1) (thickness 0.15)))
     )
@@
       (effects (font (size 1 1) (thickness 0.15)))
     )
-    (fp_text value "Conn_01x02" (at 0 4.87) (layer "F.Fab")
+    (fp_text value "PH1-02-UA" (at 0 4.87) (layer "F.Fab")
       (effects (font (size 1 1) (thickness 0.15)))
     )
@@
       (effects (font (size 1 1) (thickness 0.15)))
     )
-    (fp_text value "Conn_02x20_Odd_Even" (at 6.096 51.181) (layer "F.Fab")
-      (effects (font (size 1 1) (thickness 0.15)))
-    )
+    (fp_text value "SSQ-120-03-F-D" (at 6.096 51.181) (layer "F.Fab")
+      (effects (font (size 1 1) (thickness 0.15)))
+    )
