File: Payload/ColoradoCUBE_Payload/DEBUG_INTERFACE.kicad_sch (KiCad schematic)
At the start: 8 parts, among them J2 Generic_Conn_01x05

Commit message: updates
Parts:
- J2: value Generic_Conn_01x05 -> PH1-05-UA
Changed lines of the file:
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@@
       (effects (font (size 1.27 1.27)) (justify left))
     )
-    (property "Value" "Generic_Conn_01x05" (id 1) (at 146.05 93.9799 0)
+    (property "Value" "PH1-05-UA" (id 1) (at 146.05 93.9799 0)
       (effects (font (size 1.27 1.27)) (justify left))
     )
