File: Payload/ColoradoCUBE_Payload/Interboard_connector.kicad_sch (KiCad schematic)
At the start: 1 part, among them J1 Conn_02x20_Odd_Even

Commit message: updates
Parts:
- J1: value Conn_02x20_Odd_Even -> SSQ-120-03-F-D
Changed lines of the file:
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@@
     (in_bom yes) (on_board yes) (fields_autoplaced)
     (property "Reference" "J1" (id 0) (at 124.46 57.15 0))
-    (property "Value" "Conn_02x20_Odd_Even" (id 1) (at 124.46 59.69 0))
+    (property "Value" "SSQ-120-03-F-D" (id 1) (at 124.46 59.69 0))
     (property "Footprint" "Connector_PinHeader_2.54mm:PinHeader_2x20_P2.54mm_Vertical" (id 2) (at 123.19 86.36 0)
       (effects (font (size 1.27 1.27)) hide)
