File: Payload/ColoradoCUBE_Payload/Temperature_Sensor.kicad_sch (KiCad schematic)
At the start: 4 parts, among them J3 Conn_01x06, J4 Conn_01x04, U2 SHT40-AD1B-R2

Commit message: updates
Parts:
- J3: value Conn_01x06 -> PR20206VBNN
- J4: value Conn_01x04 -> PR20204VBNN
Changed lines of the file:
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@@
       (effects (font (size 1.27 1.27)) (justify left))
     )
-    (property "Value" "Conn_01x06" (id 1) (at 186.055 79.3749 0)
+    (property "Value" "PR20206VBNN" (id 1) (at 186.055 79.3749 0)
       (effects (font (size 1.27 1.27)) (justify left))
     )
@@
       (effects (font (size 1.27 1.27)) (justify left))
     )
-    (property "Value" "Conn_01x04" (id 1) (at 220.345 78.1049 0)
+    (property "Value" "PR20204VBNN" (id 1) (at 220.345 78.1049 0)
       (effects (font (size 1.27 1.27)) (justify left))
     )
